Commit message: Almost fixed: Adjusted controller PIDs

File: rosstuff/catkin_ws/src/arm_1v2_description/urdf/arm_1v2.xacro (robot description, xacro)
@@ -4,9 +4,11 @@
 <xacro:include filename="$(find arm_1v2_description)/urdf/arm_1v2.trans" />
 <xacro:include filename="$(find arm_1v2_description)/urdf/arm_1v2.gazebo" />
+<link name="dummy">
+</link>
 <link name="base_link">
   <inertial>
     <origin rpy="0 0 0" xyz="0.039996602784261225 0.040054601126102964 0.004961008287480484"/>
-    <mass value="0.4968646843052768"/>
-    <inertia ixx="0.000271" ixy="-0.0" ixz="0.0" iyy="0.000272" iyz="-0.0" izz="0.000534"/>
+    <mass value="10.00"/>
+    <inertia ixx="0.000" ixy="-0.0" ixz="0.0" iyy="0.000" iyz="-0.0" izz="0.000"/>
   </inertial>
   <visual>
@@ -164,4 +166,8 @@
   </collision>
 </link>
+<joint name="dummy_joint" type="fixed">
+    <parent link="dummy"/>
+    <child link="base_link"/>
+</joint>
 <joint name="Rigid1" type="fixed">
   <origin rpy="0 0 0" xyz="0.047 0.0211 0.007"/>

Commit message: Fixed URDF files: However, yaml file needs work, too jittery

File: rosstuff/catkin_ws/src/arm_1v2_description/urdf/arm_1v2.xacro (robot description, xacro)
@@ -4,12 +4,7 @@
 <xacro:include filename="$(find arm_1v2_description)/urdf/arm_1v2.trans" />
 <xacro:include filename="$(find arm_1v2_description)/urdf/arm_1v2.gazebo" />
-<link name="dummy">
+<link name="world">
 </link>
 <link name="base_link">
-  <inertial>
-    <origin rpy="0 0 0" xyz="0.039996602784261225 0.040054601126102964 0.004961008287480484"/>
-    <mass value="10.00"/>
-    <inertia ixx="0.000" ixy="-0.0" ixz="0.0" iyy="0.000" iyz="-0.0" izz="0.000"/>
-  </inertial>
   <visual>
     <origin rpy="0 0 0" xyz="0 0 0"/>
@@ -166,6 +161,6 @@
   </collision>
 </link>
-<joint name="dummy_joint" type="fixed">
-    <parent link="dummy"/>
+<joint name="ground" type="fixed">
+    <parent link="world"/>
     <child link="base_link"/>
 </joint>
