Commit message: Modified stubby_v2 and stubby controller to controm the stubby_v2

File: rosstuff/catkin_ws/src/stubby_v2_description/urdf/stubby_v2.xacro (robot description, xacro)
@@ -4,4 +4,6 @@
 <xacro:include filename="$(find stubby_v2_description)/urdf/stubby_v2.trans" />
 <xacro:include filename="$(find stubby_v2_description)/urdf/stubby_v2.gazebo" />
+<link name="world">
+</link>
 <link name="base_link">
   <inertial>
@@ -264,4 +266,13 @@
   </collision>
 </link>
+<gazebo>
+    <plugin name="gazebo_ros_control" filename="libgazebo_ros_control.so">
+        <robotNamespace>/stubby_v2</robotNamespace>
+    </plugin>
+</gazebo>
+<joint name="worldLink" type="fixed">
+    <parent link="world"/>
+    <child link="base_link"/>
+</joint>
 <joint name="Rev1" type="continuous">
   <origin rpy="0 0 0" xyz="0.0 0.0 0.037"/>
