Commit message: Updated stubby_complete

File: rosstuff/catkin_ws/src/stubby_complete_description/urdf/stubby_complete.xacro (robot description, xacro)
@@ -4,4 +4,6 @@
 <xacro:include filename="$(find stubby_complete_description)/urdf/stubby_complete.trans" />
 <xacro:include filename="$(find stubby_complete_description)/urdf/stubby_complete.gazebo" />
+<link name="world">
+</link>
 <link name="base_link">
   <inertial>
@@ -424,4 +426,13 @@
   </collision>
 </link>
+<gazebo>
+    <plugin name="gazebo_ros_control" filename="libgazebo_ros_control.so">
+        <robotNamespace>stubby_complete</robotNamespace>
+    </plugin>
+</gazebo>
+<joint name="world_link" type="fixed">
+    <parent link="world"/>
+    <child link="base_link"/>
+</joint>
 <joint name="yaw" type="continuous">
   <origin rpy="0 0 0" xyz="0.0 0.0 0.037"/>

Commit message: Added hopefully the last model

File: rosstuff/catkin_ws/src/stubby_complete_description/urdf/stubby_complete.xacro (robot description, xacro)
@@ -4,11 +4,9 @@
 <xacro:include filename="$(find stubby_complete_description)/urdf/stubby_complete.trans" />
 <xacro:include filename="$(find stubby_complete_description)/urdf/stubby_complete.gazebo" />
-<link name="world">
-</link>
 <link name="base_link">
   <inertial>
-    <origin rpy="0 0 0" xyz="-0.0946351884902972 -0.08390729542541507 0.029949542350383874"/>
-    <mass value="2.9540424862254815"/>
-    <inertia ixx="0.021201" ixy="0.0" ixz="-0.0" iyy="0.010579" iyz="-6.6e-05" izz="0.030285"/>
+    <origin rpy="0 0 0" xyz="-0.09999999999999991 -0.020966127283006095 0.021818497006580385"/>
+    <mass value="2.9547595128701887"/>
+    <inertia ixx="0.021203" ixy="-0.0" ixz="-0.0" iyy="0.010579" iyz="-6.5e-05" izz="0.030287"/>
   </inertial>
   <visual>
@@ -26,12 +24,52 @@
   </collision>
 </link>
+<link name="Component1_1">
+  <inertial>
+    <origin rpy="0 0 0" xyz="-0.04000000000451927 -0.03980214384253428 0.008090034598972902"/>
+    <mass value="0.4759246467338889"/>
+    <inertia ixx="0.000408" ixy="0.0" ixz="0.0" iyy="0.000441" iyz="-0.0" izz="0.000831"/>
+  </inertial>
+  <visual>
+    <origin rpy="0 0 0" xyz="0.06 0.026523 -0.045914"/>
+    <geometry>
+      <mesh filename="package://stubby_complete_description/meshes/Component1_1.stl" scale="0.001 0.001 0.001"/>
+    </geometry>
+    <material name="silver"/>
+  </visual>
+  <collision>
+    <origin rpy="0 0 0" xyz="0.06 0.026523 -0.045914"/>
+    <geometry>
+      <mesh filename="package://stubby_complete_description/meshes/Component1_1.stl" scale="0.001 0.001 0.001"/>
+    </geometry>
+  </collision>
+</link>
+<link name="Component2_1">
+  <inertial>
+    <origin rpy="0 0 0" xyz="-3.1092385663913924e-05 -0.012761856959488546 0.017058190511466446"/>
+    <mass value="0.04244091097100989"/>
+    <inertia ixx="1.2e-05" ixy="-0.0" ixz="0.0" iyy="7e-06" iyz="-0.0" izz="1e-05"/>
+  </inertial>
+  <visual>
+    <origin rpy="0 0 0" xyz="0.1 0.052023 -0.060914"/>
+    <geometry>
+      <mesh filename="package://stubby_complete_description/meshes/Component2_1.stl" scale="0.001 0.001 0.001"/>
+    </geometry>
+    <material name="silver"/>
+  </visual>
+  <collision>
+    <origin rpy="0 0 0" xyz="0.1 0.052023 -0.060914"/>
+    <geometry>
+      <mesh filename="package://stubby_complete_description/meshes/Component2_1.stl" scale="0.001 0.001 0.001"/>
+    </geometry>
+  </collision>
+</link>
 <link name="Component3_1">
   <inertial>
-    <origin rpy="0 0 0" xyz="-3.222924193166388e-05 1.950762713864851e-07 0.0023373639782219707"/>
+    <origin rpy="0 0 0" xyz="-3.2040751634265785e-05 4.2101147429418617e-07 0.002337181396787208"/>
     <mass value="0.02417691266422109"/>
     <inertia ixx="1e-06" ixy="-0.0" ixz="-0.0" iyy="4e-06" iyz="-0.0" izz="5e-06"/>
   </inertial>
   <visual>
-    <origin rpy="0 0 0" xyz="0.094635 0.119475 -0.104052"/>
+    <origin rpy="0 0 0" xyz="0.1 0.052023 -0.097914"/>
     <geometry>
       <mesh filename="package://stubby_complete_description/meshes/Component3_1.stl" scale="0.001 0.001 0.001"/>
@@ -40,5 +78,5 @@
   </visual>
   <collision>
-    <origin rpy="0 0 0" xyz="0.094635 0.119475 -0.104052"/>
+    <origin rpy="0 0 0" xyz="0.1 0.052023 -0.097914"/>
     <geometry>
       <mesh filename="package://stubby_complete_description/meshes/Component3_1.stl" scale="0.001 0.001 0.001"/>
@@ -46,101 +84,21 @@
   </collision>
 </link>
-<link name="Component4__1">
-  <inertial>
-    <origin rpy="0 0 0" xyz="-0.014941605750908832 0.001737917105307435 0.01353088273917584"/>
+<link name="Component4_1">
+  <inertial>
+    <origin rpy="0 0 0" xyz="-0.01494141726061049 -0.006261856959488575 0.013530700157741146"/>
     <mass value="0.04244091097100989"/>
     <inertia ixx="1e-05" ixy="-0.0" ixz="-0.0" iyy="7e-06" iyz="0.0" izz="1.2e-05"/>
   </inertial>
   <visual>
-    <origin rpy="0 0 0" xyz="0.078635 0.119475 -0.109552"/>
-    <geometry>
-      <mesh filename="package://stubby_complete_description/meshes/Component4__1.stl" scale="0.001 0.001 0.001"/>
-    </geometry>
-    <material name="silver"/>
-  </visual>
-  <collision>
-    <origin rpy="0 0 0" xyz="0.078635 0.119475 -0.109552"/>
-    <geometry>
-      <mesh filename="package://stubby_complete_description/meshes/Component4__1.stl" scale="0.001 0.001 0.001"/>
-    </geometry>
-  </collision>
-</link>
-<link name="Component1_1">
-  <inertial>
-    <origin rpy="0 0 0" xyz="-2.7950320549557928e-06 4.208824011434076e-05 0.006457052192550834"/>
-    <mass value="0.6475846843052765"/>
-    <inertia ixx="0.000356" ixy="-0.0" ixz="0.0" iyy="0.000357" iyz="-0.0" izz="0.000695"/>
-  </inertial>
-  <visual>
-    <origin rpy="0 0 0" xyz="0.094635 0.129475 -0.054052"/>
-    <geometry>
-      <mesh filename="package://stubby_complete_description/meshes/Component1_1.stl" scale="0.001 0.001 0.001"/>
-    </geometry>
-    <material name="silver"/>
-  </visual>
-  <collision>
-    <origin rpy="0 0 0" xyz="0.094635 0.129475 -0.054052"/>
-    <geometry>
-      <mesh filename="package://stubby_complete_description/meshes/Component1_1.stl" scale="0.001 0.001 0.001"/>
-    </geometry>
-  </collision>
-</link>
-<link name="Component2_1">
-  <inertial>
-    <origin rpy="0 0 0" xyz="-3.128087596129814e-05 -0.012762082894690802 0.017058373092900925"/>
-    <mass value="0.04244091097100989"/>
-    <inertia ixx="1.2e-05" ixy="-0.0" ixz="0.0" iyy="7e-06" iyz="-0.0" izz="1e-05"/>
-  </inertial>
-  <visual>
-    <origin rpy="0 0 0" xyz="0.094635 0.119475 -0.067052"/>
-    <geometry>
-      <mesh filename="package://stubby_complete_description/meshes/Component2_1.stl" scale="0.001 0.001 0.001"/>
-    </geometry>
-    <material name="silver"/>
-  </visual>
-  <collision>
-    <origin rpy="0 0 0" xyz="0.094635 0.119475 -0.067052"/>
-    <geometry>
-      <mesh filename="package://stubby_complete_description/meshes/Component2_1.stl" scale="0.001 0.001 0.001"/>
-    </geometry>
-  </collision>
-</link>
-<link name="platform1_1">
-  <inertial>
-    <origin rpy="0 0 0" xyz="-1.8849029877199275e-07 0.00020232718072946826 0.0049935033993906"/>
-    <mass value="0.4507941946898463"/>
-    <inertia ixx="0.001622" ixy="-0.0" ixz="0.0" iyy="0.001632" iyz="-0.0" izz="0.003247"/>
-  </inertial>
-  <visual>
-    <origin rpy="0 0 0" xyz="0.094635 -0.060525 -0.054052"/>
-    <geometry>
-      <mesh filename="package://stubby_complete_description/meshes/platform1_1.stl" scale="0.001 0.001 0.001"/>
-    </geometry>
-    <material name="silver"/>
-  </visual>
-  <collision>
-    <origin rpy="0 0 0" xyz="0.094635 -0.060525 -0.054052"/>
-    <geometry>
-      <mesh filename="package://stubby_complete_description/meshes/platform1_1.stl" scale="0.001 0.001 0.001"/>
-    </geometry>
-  </collision>
-</link>
-<link name="susMount1_1">
-  <inertial>
-    <origin rpy="0 0 0" xyz="-0.017788026341239802 0.26356555152104366 0.18981987323024652"/>
-    <mass value="0.6557743433400158"/>
-    <inertia ixx="0.001646" ixy="-0.0" ixz="-4e-06" iyy="0.001645" iyz="1e-05" izz="5.2e-05"/>
-  </inertial>
-  <visual>
-    <origin rpy="0 0 0" xyz="-0.01073 0.333527 0.015723"/>
-    <geometry>
-      <mesh filename="package://stubby_complete_description/meshes/susMount1_1.stl" scale="0.001 0.001 0.001"/>
-    </geometry>
-    <material name="silver"/>
-  </visual>
-  <collision>
-    <origin rpy="0 0 0" xyz="-0.01073 0.333527 0.015723"/>
-    <geometry>
-      <mesh filename="package://stubby_complete_description/meshes/susMount1_1.stl" scale="0.001 0.001 0.001"/>
+    <origin rpy="0 0 0" xyz="0.084 0.044023 -0.103414"/>
+    <geometry>
+      <mesh filename="package://stubby_complete_description/meshes/Component4_1.stl" scale="0.001 0.001 0.001"/>
+    </geometry>
+    <material name="silver"/>
+  </visual>
+  <collision>
+    <origin rpy="0 0 0" xyz="0.084 0.044023 -0.103414"/>
+    <geometry>
+      <mesh filename="package://stubby_complete_description/meshes/Component4_1.stl" scale="0.001 0.001 0.001"/>
     </geometry>
   </collision>
@@ -148,10 +106,10 @@
 <link name="Component5_1">
   <inertial>
-    <origin rpy="0 0 0" xyz="0.0003232513687730365 0.04421280486587253 1.034989279184717e-05"/>
+    <origin rpy="0 0 0" xyz="0.000323439859071295 0.044213030801076594 1.0167311355765984e-05"/>
     <mass value="0.07320231395363634"/>
     <inertia ixx="8e-05" ixy="4e-06" ixz="0.0" iyy="6e-06" iyz="-0.0" izz="7.5e-05"/>
   </inertial>
   <visual>
-    <origin rpy="0 0 0" xyz="0.073635 0.104975 -0.123052"/>
+    <origin rpy="0 0 0" xyz="0.079 0.037523 -0.116914"/>
     <geometry>
       <mesh filename="package://stubby_complete_description/meshes/Component5_1.stl" scale="0.001 0.001 0.001"/>
@@ -160,5 +118,5 @@
   </visual>
   <collision>
-    <origin rpy="0 0 0" xyz="0.073635 0.104975 -0.123052"/>
+    <origin rpy="0 0 0" xyz="0.079 0.037523 -0.116914"/>
     <geometry>
       <mesh filename="package://stubby_complete_description/meshes/Component5_1.stl" scale="0.001 0.001 0.001"/>
@@ -166,72 +124,92 @@
   </collision>
 </link>
-<link name="Component6__1">
-  <inertial>
-    <origin rpy="0 0 0" xyz="-0.01494160575090872 0.017737917105307355 -0.01346911726082041"/>
+<link name="Component6_1">
+  <inertial>
+    <origin rpy="0 0 0" xyz="-0.01494141726061049 0.01773814304051132 -0.013469299842258711"/>
     <mass value="0.04244091097100989"/>
     <inertia ixx="1e-05" ixy="-0.0" ixz="-0.0" iyy="7e-06" iyz="0.0" izz="1.2e-05"/>
   </inertial>
   <visual>
-    <origin rpy="0 0 0" xyz="0.078635 0.015475 -0.136552"/>
-    <geometry>
-      <mesh filename="package://stubby_complete_description/meshes/Component6__1.stl" scale="0.001 0.001 0.001"/>
-    </geometry>
-    <material name="silver"/>
-  </visual>
-  <collision>
-    <origin rpy="0 0 0" xyz="0.078635 0.015475 -0.136552"/>
-    <geometry>
-      <mesh filename="package://stubby_complete_description/meshes/Component6__1.stl" scale="0.001 0.001 0.001"/>
-    </geometry>
-  </collision>
-</link>
-<link name="LEFT1_1">
-  <inertial>
-    <origin rpy="0 0 0" xyz="-0.0037516937714175413 -0.03733422612574102 -0.007881515172349696"/>
-    <mass value="0.08018389659681822"/>
-    <inertia ixx="9.5e-05" ixy="-3e-06" ixz="-0.0" iyy="7e-06" iyz="-0.0" izz="8.8e-05"/>
-  </inertial>
-  <visual>
-    <origin rpy="0 0 0" xyz="0.110635 0.020975 -0.131052"/>
-    <geometry>
-      <mesh filename="package://stubby_complete_description/meshes/LEFT1_1.stl" scale="0.001 0.001 0.001"/>
-    </geometry>
-    <material name="silver"/>
-  </visual>
-  <collision>
-    <origin rpy="0 0 0" xyz="0.110635 0.020975 -0.131052"/>
-    <geometry>
-      <mesh filename="package://stubby_complete_description/meshes/LEFT1_1.stl" scale="0.001 0.001 0.001"/>
-    </geometry>
-  </collision>
-</link>
-<link name="Component9_1">
-  <inertial>
-    <origin rpy="0 0 0" xyz="0.00032325136877307814 0.04421280486587255 1.0349892795746829e-05"/>
+    <origin rpy="0 0 0" xyz="0.084 -0.051977 -0.130414"/>
+    <geometry>
+      <mesh filename="package://stubby_complete_description/meshes/Component6_1.stl" scale="0.001 0.001 0.001"/>
+    </geometry>
+    <material name="silver"/>
+  </visual>
+  <collision>
+    <origin rpy="0 0 0" xyz="0.084 -0.051977 -0.130414"/>
+    <geometry>
+      <mesh filename="package://stubby_complete_description/meshes/Component6_1.stl" scale="0.001 0.001 0.001"/>
+    </geometry>
+  </collision>
+</link>
+<link name="Component7_1">
+  <inertial>
+    <origin rpy="0 0 0" xyz="-0.003787166400802497 -0.03908271518949953 -0.013398484021248727"/>
+    <mass value="0.05604795467246254"/>
+    <inertia ixx="4.5e-05" ixy="-1e-06" ixz="-0.0" iyy="4e-06" iyz="-0.0" izz="4.1e-05"/>
+  </inertial>
+  <visual>
+    <origin rpy="0 0 0" xyz="0.116 -0.051977 -0.130414"/>
+    <geometry>
+      <mesh filename="package://stubby_complete_description/meshes/Component7_1.stl" scale="0.001 0.001 0.001"/>
+    </geometry>
+    <material name="silver"/>
+  </visual>
+  <collision>
+    <origin rpy="0 0 0" xyz="0.116 -0.051977 -0.130414"/>
+    <geometry>
+      <mesh filename="package://stubby_complete_description/meshes/Component7_1.stl" scale="0.001 0.001 0.001"/>
+    </geometry>
+  </collision>
+</link>
+<link name="Component8_1">
+  <inertial>
+    <origin rpy="0 0 0" xyz="0.00032343985907133666 0.04421303080107655 1.0167311355960273e-05"/>
     <mass value="0.07320231395363634"/>
     <inertia ixx="8e-05" ixy="4e-06" ixz="0.0" iyy="6e-06" iyz="-0.0" izz="7.5e-05"/>
   </inertial>
   <visual>
-    <origin rpy="0 0 0" xyz="0.073635 -0.015025 -0.123052"/>
-    <geometry>
-      <mesh filename="package://stubby_complete_description/meshes/Component9_1.stl" scale="0.001 0.001 0.001"/>
-    </geometry>
-    <material name="silver"/>
-  </visual>
-  <collision>
-    <origin rpy="0 0 0" xyz="0.073635 -0.015025 -0.123052"/>
-    <geometry>
-      <mesh filename="package://stubby_complete_description/meshes/Component9_1.stl" scale="0.001 0.001 0.001"/>
-    </geometry>
-  </collision>
-</link>
-<link name="Component10_1">
-  <inertial>
-    <origin rpy="0 0 0" xyz="-0.01494160575090872 0.017737917105307255 -0.013469117260816538"/>
+    <origin rpy="0 0 0" xyz="0.079 -0.082477 -0.116914"/>
+    <geometry>
+      <mesh filename="package://stubby_complete_description/meshes/Component8_1.stl" scale="0.001 0.001 0.001"/>
+    </geometry>
+    <material name="silver"/>
+  </visual>
+  <collision>
+    <origin rpy="0 0 0" xyz="0.079 -0.082477 -0.116914"/>
+    <geometry>
+      <mesh filename="package://stubby_complete_description/meshes/Component8_1.stl" scale="0.001 0.001 0.001"/>
+    </geometry>
+  </collision>
+</link>
+<link name="Component9_1">
+  <inertial>
+    <origin rpy="0 0 0" xyz="-0.014941417260610448 0.017738143040511356 -0.01346929984225867"/>
     <mass value="0.04244091097100989"/>
     <inertia ixx="1e-05" ixy="-0.0" ixz="-0.0" iyy="7e-06" iyz="0.0" izz="1.2e-05"/>
   </inertial>
   <visual>
-    <origin rpy="0 0 0" xyz="0.078635 -0.104525 -0.136552"/>
+    <origin rpy="0 0 0" xyz="0.084 -0.171977 -0.130414"/>
+    <geometry>
+      <mesh filename="package://stubby_complete_description/meshes/Component9_1.stl" scale="0.001 0.001 0.001"/>
+    </geometry>
+    <material name="silver"/>
+  </visual>
+  <collision>
+    <origin rpy="0 0 0" xyz="0.084 -0.171977 -0.130414"/>
+    <geometry>
+      <mesh filename="package://stubby_complete_description/meshes/Component9_1.stl" scale="0.001 0.001 0.001"/>
+    </geometry>
+  </collision>
+</link>
+<link name="Component10_1">
+  <inertial>
+    <origin rpy="0 0 0" xyz="-0.0037871664008025108 -0.03908271518949957 -0.013398484021248672"/>
+    <mass value="0.05604795467246254"/>
+    <inertia ixx="4.5e-05" ixy="-1e-06" ixz="-0.0" iyy="4e-06" iyz="-0.0" izz="4.1e-05"/>
+  </inertial>
+  <visual>
+    <origin rpy="0 0 0" xyz="0.116 -0.171977 -0.130414"/>
     <geometry>
       <mesh filename="package://stubby_complete_description/meshes/Component10_1.stl" scale="0.001 0.001 0.001"/>
@@ -240,5 +218,5 @@
   </visual>
   <collision>
-    <origin rpy="0 0 0" xyz="0.078635 -0.104525 -0.136552"/>
+    <origin rpy="0 0 0" xyz="0.116 -0.171977 -0.130414"/>
     <geometry>
       <mesh filename="package://stubby_complete_description/meshes/Component10_1.stl" scale="0.001 0.001 0.001"/>
@@ -246,32 +224,12 @@
   </collision>
 </link>
-<link name="LEFT2_1">
-  <inertial>
-    <origin rpy="0 0 0" xyz="-0.0037516937210517326 -0.0508342261257418 -0.013381515214388101"/>
-    <mass value="0.0801838965968182"/>
-    <inertia ixx="9.5e-05" ixy="-3e-06" ixz="-0.0" iyy="7e-06" iyz="-0.0" izz="8.8e-05"/>
-  </inertial>
-  <visual>
-    <origin rpy="0 0 0" xyz="0.110635 -0.112525 -0.136552"/>
-    <geometry>
-      <mesh filename="package://stubby_complete_description/meshes/LEFT2_1.stl" scale="0.001 0.001 0.001"/>
-    </geometry>
-    <material name="silver"/>
-  </visual>
-  <collision>
-    <origin rpy="0 0 0" xyz="0.110635 -0.112525 -0.136552"/>
-    <geometry>
-      <mesh filename="package://stubby_complete_description/meshes/LEFT2_1.stl" scale="0.001 0.001 0.001"/>
-    </geometry>
-  </collision>
-</link>
 <link name="Component11_1">
   <inertial>
-    <origin rpy="0 0 0" xyz="-0.021000188161351227 0.025472256393286846 -0.00021028594488545216"/>
-    <mass value="0.08541239044327154"/>
-    <inertia ixx="2.6e-05" ixy="-0.0" ixz="-0.0" iyy="4.2e-05" iyz="0.0" izz="5.6e-05"/>
-  </inertial>
-  <visual>
-    <origin rpy="0 0 0" xyz="0.073635 -0.135025 -0.123052"/>
+    <origin rpy="0 0 0" xyz="-0.021096269692649494 0.02403068850135351 -0.0008093901396380859"/>
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